File: pcb/UCB_board.kicad_sch (KiCad schematic)
At the start: 28 parts

Commit message: PartNumber update
Parts:
- D1, D13, D14, D2, D4, D6: Manufacturer_Part_Number (none) -> FYLS-1206PGC
- R23, R24, R25, R26: Manufacturer_Part_Number (none) -> CRCW04020000Z0TDBC
- R86, R87: Manufacturer_Part_Number (none) -> 0603SAF1200T5E
- RN1: Manufacturer_Part_Number (none) -> 4D03WGJ0103T5E
Changed lines of the file:
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@@
+			)
+		)
+		(property "Manufacturer_Part_Number" "FYLS-1206PGC "
+			(at 151.13 137.16 90)
+			(effects
+				(font
+					(size 1.27 1.27)
+				)
+				(hide yes)
 			)
 		)
@@
 			)
 		)
+		(property "Manufacturer_Part_Number" "CRCW04020000Z0TDBC "
+			(at 179.07 46.99 90)
+			(effects
+				(font
+					(size 1.27 1.27)
+				)
+				(hide yes)
+			)
+		)
 		(pin "1"
 		)
@@
 			)
 		)
+		(property "Manufacturer_Part_Number" "FYLS-1206PGC "
+			(at 77.47 123.19 90)
+			(effects
+				(font
+					(size 1.27 1.27)
+				)
+				(hide yes)
+			)
+		)
 		(pin "1"
 		)
@@
 		(property "Sim.Pins" "1=K 2=A"
 			(at 67.31 123.19 0)
+			(effects
+				(font
+					(size 1.27 1.27)
+				)
+				(hide yes)
+			)
+		)
+		(property "Manufacturer_Part_Number" "FYLS-1206PGC "
+			(at 67.31 123.19 90)
 			(effects
 				(font
@@
 			)
 		)
+		(property "Manufacturer_Part_Number" "CRCW04020000Z0TDBC "
+			(at 179.07 41.91 90)
+			(effects
+				(font
+					(size 1.27 1.27)
+				)
+				(hide yes)
+			)
+		)
 		(pin "1"
 		)
@@
 			)
 		)
+		(property "Manufacturer_Part_Number" "0603SAF1200T5E "
+			(at 67.31 132.08 0)
+			(effects
+				(font
+					(size 1.27 1.27)
+				)
+				(hide yes)
+			)
+		)
 		(pin "1"
 		)
@@
 			)
 		)
+		(property "Manufacturer_Part_Number" "CRCW04020000Z0TDBC "
+			(at 179.07 49.53 90)
+			(effects
+				(font
+					(size 1.27 1.27)
+				)
+				(hide yes)
+			)
+		)
 		(pin "1"
 		)
@@
 		(property "Description" "4D03WGJ0103T5E"
 			(at 153.67 149.86 0)
+			(effects
+				(font
+					(size 1.27 1.27)
+				)
+				(hide yes)
+			)
+		)
+		(property "Manufacturer_Part_Number" "4D03WGJ0103T5E"
+			(at 153.67 149.86 90)
 			(effects
 				(font
@@
 			)
 		)
+		(property "Manufacturer_Part_Number" "0603SAF1200T5E "
+			(at 77.47 132.08 0)
+			(effects
+				(font
+					(size 1.27 1.27)
+				)
+				(hide yes)
+			)
+		)
 		(pin "1"
 		)
@@
 			)
 		)
+		(property "Manufacturer_Part_Number" "FYLS-1206PGC "
+			(at 166.37 137.16 90)
+			(effects
+				(font
+					(size 1.27 1.27)
+				)
+				(hide yes)
+			)
+		)
 		(pin "1"
 		)
@@
 			)
 		)
+		(property "Manufacturer_Part_Number" "FYLS-1206PGC "
+			(at 143.51 137.16 90)
+			(effects
+				(font
+					(size 1.27 1.27)
+				)
+				(hide yes)
+			)
+		)
 		(pin "1"
 		)
@@
 		(property "Sim.Pins" "1=K 2=A"
 			(at 158.75 137.16 0)
+			(effects
+				(font
+					(size 1.27 1.27)
+				)
+				(hide yes)
+			)
+		)
+		(property "Manufacturer_Part_Number" "FYLS-1206PGC "
+			(at 158.75 137.16 90)
 			(effects
 				(font
@@
 			(effects
 				(font
+					(size 1.27 1.27)
+				)
+				(hide yes)
+			)
+		)
+		(property "Manufacturer_Part_Number" "CRCW04020000Z0TDBC "
+			(at 179.07 44.45 90)
+			(effects
+				(font
