File: pcb/MCU.kicad_sch (KiCad schematic)
At the start: 28 parts, among them J2 TC2030, J3 Conn_01x02_Pin, U2 LM4040DBZ-3, U6 FM24C64B, U7 STM32H563VITx, Y1 3225-25M-SR

Commit message: PartNumber update
Parts:
- C27: Manufacturer_Part_Number (none) -> GRM1885C1H103JA01J
- C29, C35, C39, C49, C50, C53, C54, C55, C58: Manufacturer_Part_Number (none) -> GRM188R71H104KA93D
- C51: Manufacturer_Part_Number (none) -> CL31B106KBHNNNE
- C56, C57: Manufacturer_Part_Number (none) -> 0603X475K100CT
- R20: footprint Resistor_SMD:R_0402_1005Metric_Pad0.72x0.64mm_HandSolder -> Resistor_SMD:R_0603_1608Metric; Manufacturer_Part_Number (none) -> 0603SAF1004T5E
- R21, R84, R85: Manufacturer_Part_Number (none) -> CRCW060310K0FKTABC
- R80: Manufacturer_Part_Number (none) -> CRCW04020000Z0TDBC
- U2: Manufacturer_Part_Number (none) -> LM4040DBZ-3
- U6: Manufacturer_Part_Number (none) -> FM24C64B
- U7: Manufacturer_Part_Number (none) -> STM32H563VIT6

Commit message: Cleaning
Changed lines of the file:
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@@
 (kicad_sch
-	(version 20250114)
+	(version 20260306)
 	(generator "eeschema")
-	(generator_version "9.0")
+	(generator_version "10.0")
 	(paper "A3")
 	(title_block
