File: pcb/ConnDIN41612.kicad_sch (KiCad schematic)
At the start: 46 parts, among them IC1 SN65HVD75DR, J1 DIN41612_02x32_AC, T1 H1102NL, U3 USBLC6-2SC6, U4 USBLC6-2SC6, U5 USBLC6-2SC6

Commit message: PartNumber update
Parts:
- C1, C2, C52: Manufacturer_Part_Number (none) -> GRM188R71H104KA93D
- C3, C5: Manufacturer_Part_Number (none) -> 1206B102K202
- C4, C7: Manufacturer_Part_Number (none) -> GRM1885C1H103JA01J
- D16, D17, D3, D5: Manufacturer_Part_Number (none) -> ESD5Z3.3T1G
- D7: Manufacturer_Part_Number (none) -> SMF5.0CA
- FB1, FB2: Manufacturer_Part_Number (none) -> WLBD1608HCU101TL
- J1: now left out of the parts list
- R1, R2: Manufacturer_Part_Number (none) -> 0402WGJ0220TCE
- R10, R11: Manufacturer_Part_Number (none) -> CRCW060349R9FKTABC
- R12, R13: Manufacturer_Part_Number (none) -> 1-2176339-5
- R3, R90, R91: Manufacturer_Part_Number (none) -> CRCW060310K0FKTABC
- R4: Manufacturer_Part_Number (none) -> RC0603FR-0715KL
- R6, R7: Manufacturer_Part_Number (none) -> 0603SAJ0750T5E
- R8, R9: Manufacturer_Part_Number (none) -> RC0603JR-0782RL
- U3, U4, U5: Manufacturer_Part_Number (none) -> USBLC6-2SC6

Commit message: Unify component values/footprints per checklist; add via-in-pad DRC rule; regenerate production outputs
Parts:
- C1, C2, C4, C52, C7: footprint Capacitor_SMD:C_0603_1608Metric_Pad1.08x0.95mm_HandSolder -> Capacitor_SMD:C_0603_1608Metric
- C3, C5: footprint Capacitor_SMD:C_1206_3216Metric_Pad1.33x1.80mm_HandSolder -> Capacitor_SMD:C_1206_3216Metric
- C73, C74: value 6,8n -> 6.8n; footprint Capacitor_SMD:C_0603_1608Metric_Pad1.08x0.95mm_HandSolder -> Capacitor_SMD:C_0603_1608Metric
- FB1, FB2: footprint Inductor_SMD:L_0603_1608Metric_Pad1.05x0.95mm_HandSolder -> Inductor_SMD:L_0603_1608Metric
- R1, R2: value 22R -> 22; footprint Resistor_SMD:R_0402_1005Metric_Pad0.72x0.64mm_HandSolder -> Resistor_SMD:R_0402_1005Metric
- R10, R11: value 49R9 -> 49.9; footprint Resistor_SMD:R_0603_1608Metric_Pad0.98x0.95mm_HandSolder -> Resistor_SMD:R_0603_1608Metric
- R12, R13: value 150R -> 150; footprint Resistor_SMD:R_0603_1608Metric_Pad0.98x0.95mm_HandSolder -> Resistor_SMD:R_0603_1608Metric
- R3, R4, R90, R91: footprint Resistor_SMD:R_0603_1608Metric_Pad0.98x0.95mm_HandSolder -> Resistor_SMD:R_0603_1608Metric
- R5, R88, R89: value 10R -> 10; footprint Resistor_SMD:R_0603_1608Metric_Pad0.98x0.95mm_HandSolder -> Resistor_SMD:R_0603_1608Metric
- R6, R7: value 75R -> 75; footprint Resistor_SMD:R_0603_1608Metric_Pad0.98x0.95mm_HandSolder -> Resistor_SMD:R_0603_1608Metric
- R8, R9: value 82R -> 82; footprint Resistor_SMD:R_0603_1608Metric_Pad0.98x0.95mm_HandSolder -> Resistor_SMD:R_0603_1608Metric
Changed lines of the file:
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@@
 			)
 		)
-		(property "Footprint" "Resistor_SMD:R_0603_1608Metric_Pad0.98x0.95mm_HandSolder"
+		(property "Footprint" "Resistor_SMD:R_0603_1608Metric"
 			(at 72.39 30.988 90)
 			(hide yes)
@@
 			)
 		)
-		(property "Footprint" "Capacitor_SMD:C_0603_1608Metric_Pad1.08x0.95mm_HandSolder"
+		(property "Footprint" "Capacitor_SMD:C_0603_1608Metric"
 			(at 91.1352 176.53 0)
 			(hide yes)
@@
 			)
 		)
-		(property "Value" "10R"
+		(property "Value" "10"
 			(at 91.44 134.6199 0)
 			(show_name no)
@@
 			)
 		)
-		(property "Footprint" "Resistor_SMD:R_0603_1608Metric_Pad0.98x0.95mm_HandSolder"
+		(property "Footprint" "Resistor_SMD:R_0603_1608Metric"
 			(at 87.122 133.35 90)
 			(hide yes)
@@
 			)
 		)
-		(property "Value" "49R9"
+		(property "Value" "49.9"
 			(at 82.55 134.6199 0)
 			(show_name no)
@@
 			)
 		)
-		(property "Footprint" "Resistor_SMD:R_0603_1608Metric_Pad0.98x0.95mm_HandSolder"
+		(property "Footprint" "Resistor_SMD:R_0603_1608Metric"
 			(at 78.232 133.35 90)
 			(hide yes)
@@
 			)
 		)
-		(property "Value" "82R"
+		(property "Value" "82"
 			(at 68.58 163.8299 0)
 			(show_name no)
@@
 			)
 		)
-		(property "Footprint" "Resistor_SMD:R_0603_1608Metric_Pad0.98x0.95mm_HandSolder"
+		(property "Footprint" "Resistor_SMD:R_0603_1608Metric"
 			(at 64.262 162.56 90)
 			(hide yes)
@@
 			)
 		)
-		(property "Footprint" "Resistor_SMD:R_0603_1608Metric_Pad0.98x0.95mm_HandSolder"
+		(property "Footprint" "Resistor_SMD:R_0603_1608Metric"
 			(at 56.388 95.25 90)
 			(hide yes)
@@
 			)
 		)
-		(property "Footprint" "Capacitor_SMD:C_0603_1608Metric_Pad1.08x0.95mm_HandSolder"
+		(property "Footprint" "Capacitor_SMD:C_0603_1608Metric"
 			(at 32.7152 133.35 0)
 			(hide yes)
@@
 			)
 		)
-		(property "Value" "10R"
+		(property "Value" "10"
 			(at 100.33 73.66 90)
 			(show_name no)
@@
 			)
 		)
-		(property "Footprint" "Resistor_SMD:R_0603_1608Metric_Pad0.98x0.95mm_HandSolder"
+		(property "Footprint" "Resistor_SMD:R_0603_1608Metric"
 			(at 100.33 79.248 90)
 			(hide yes)
@@
 			)
 		)
-		(property "Footprint" "Inductor_SMD:L_0603_1608Metric_Pad1.05x0.95mm_HandSolder"
+		(property "Footprint" "Inductor_SMD:L_0603_1608Metric"
 			(at 83.312 120.65 90)
 			(hide yes)
@@
 			)
 		)
-		(property "Footprint" "Capacitor_SMD:C_0603_1608Metric_Pad1.08x0.95mm_HandSolder"
+		(property "Footprint" "Capacitor_SMD:C_0603_1608Metric"
 			(at 44.1452 133.35 0)
 			(hide yes)
@@
 			)
 		)
-		(property "Value" "82R"
+		(property "Value" "82"
 			(at 76.2 163.8299 0)
 			(show_name no)
@@
 			)
 		)
-		(property "Footprint" "Resistor_SMD:R_0603_1608Metric_Pad0.98x0.95mm_HandSolder"
+		(property "Footprint" "Resistor_SMD:R_0603_1608Metric"
 			(at 71.882 162.56 90)
 			(hide yes)
@@
 			)
 		)
-		(property "Footprint" "Inductor_SMD:L_0603_1608Metric_Pad1.05x0.95mm_HandSolder"
+		(property "Footprint" "Inductor_SMD:L_0603_1608Metric"
 			(at 104.14 30.988 90)
 			(hide yes)
@@
 			)
 		)
-		(property "Value" "22R"
+		(property "Value" "22"
 			(at 57.15 36.83 90)
 			(show_name no)
@@
 			)
 		)
-		(property "Footprint" "Resistor_SMD:R_0402_1005Metric_Pad0.72x0.64mm_HandSolder"
+		(property "Footprint" "Resistor_SMD:R_0402_1005Metric"
 			(at 57.15 42.418 90)
 			(hide yes)
@@
 			)
 		)
-		(property "Value" "150R"
+		(property "Value" "150"
 			(at 140.97 167.6399 0)
 			(show_name no)
@@
 			)
 		)
-		(property "Footprint" "Resistor_SMD:R_0603_1608Metric_Pad0.98x0.95mm_HandSolder"
+		(property "Footprint" "Resistor_SMD:R_0603_1608Metric"
 			(at 136.652 166.37 90)
 			(hide yes)
@@
 			)
 		)
-		(property "Footprint" "Capacitor_SMD:C_1206_3216Metric_Pad1.33x1.80mm_HandSolder"
+		(property "Footprint" "Capacitor_SMD:C_1206_3216Metric"
 			(at 124.1552 182.88 0)
 			(hide yes)
@@
 			)
 		)
-		(property "Footprint" "Capacitor_SMD:C_0603_1608Metric_Pad1.08x0.95mm_HandSolder"
+		(property "Footprint" "Capacitor_SMD:C_0603_1608Metric"
 			(at 88.5952 73.66 0)
 			(hide yes)
@@
 			)
 		)
-		(property "Value" "6,8n"
+		(property "Value" "6.8n"
 			(at 83.82 155.702 0)
 			(show_name no)
@@
 			)
 		)
-		(property "Footprint" "Capacitor_SMD:C_0603_1608Metric_Pad1.08x0.95mm_HandSolder"
+		(property "Footprint" "Capacitor_SMD:C_0603_1608Metric"
 			(at 78.74 153.3652 0)
 			(hide yes)
@@
 			)
 		)
-		(property "Value" "150R"
+		(property "Value" "150"
 			(at 149.86 167.6399 0)
 			(show_name no)
@@
 			)
 		)
-		(property "Footprint" "Resistor_SMD:R_0603_1608Metric_Pad0.98x0.95mm_HandSolder"
+		(property "Footprint" "Resistor_SMD:R_0603_1608Metric"
 			(at 145.542 166.37 90)
 			(hide yes)
@@
 			)
 		)
-		(property "Value" "10R"
+		(property "Value" "10"
 			(at 100.33 87.63 90)
 			(show_name no)
@@
 			)
 		)
-		(property "Footprint" "Resistor_SMD:R_0603_1608Metric_Pad0.98x0.95mm_HandSolder"
+		(property "Footprint" "Resistor_SMD:R_0603_1608Metric"
 			(at 100.33 93.218 90)
 			(hide yes)
@@
 			)
 		)
-		(property "Footprint" "Resistor_SMD:R_0603_1608Metric_Pad0.98x0.95mm_HandSolder"
+		(property "Footprint" "Resistor_SMD:R_0603_1608Metric"
 			(at 62.23 30.988 90)
 			(hide yes)
@@
 			)
 		)
-		(property "Value" "22R"
+		(property "Value" "22"
 			(at 62.23 34.29 90)
 			(show_name no)
@@
 			)
 		)
-		(property "Footprint" "Resistor_SMD:R_0402_1005Metric_Pad0.72x0.64mm_HandSolder"
+		(property "Footprint" "Resistor_SMD:R_0402_1005Metric"
 			(at 62.23 39.878 90)
 			(hide yes)
@@
 			)
 		)
-		(property "Value" "49R9"
+		(property "Value" "49.9"
 			(at 73.66 134.6199 0)
 			(show_name no)
@@
 			)
 		)
-		(property "Footprint" "Resistor_SMD:R_0603_1608Metric_Pad0.98x0.95mm_HandSolder"
+		(property "Footprint" "Resistor_SMD:R_0603_1608Metric"
 			(at 69.342 133.35 90)
 			(hide yes)
@@
 			)
 		)
-		(property "Footprint" "Capacitor_SMD:C_0603_1608Metric_Pad1.08x0.95mm_HandSolder"
+		(property "Footprint" "Capacitor_SMD:C_0603_1608Metric"
 			(at 82.8548 168.91 0)
 			(hide yes)
@@
 			)
 		)
-		(property "Value" "75R"
+		(property "Value" "75"
 			(at 125.73 167.6399 0)
 			(show_name no)
@@
 			)
 		)
-		(property "Footprint" "Resistor_SMD:R_0603_1608Metric_Pad0.98x0.95mm_HandSolder"
+		(property "Footprint" "Resistor_SMD:R_0603_1608Metric"
 			(at 121.412 166.37 90)
 			(hide yes)
@@
 			)
 		)
-		(property "Value" "75R"
+		(property "Value" "75"
 			(at 133.35 167.6399 0)
 			(show_name no)
@@
 			)
 		)
-		(property "Footprint" "Resistor_SMD:R_0603_1608Metric_Pad0.98x0.95mm_HandSolder"
+		(property "Footprint" "Resistor_SMD:R_0603_1608Metric"
 			(at 129.032 166.37 90)
 			(hide yes)
@@
 			)
 		)
-		(property "Footprint" "Resistor_SMD:R_0603_1608Metric_Pad0.98x0.95mm_HandSolder"
+		(property "Footprint" "Resistor_SMD:R_0603_1608Metric"
 			(at 56.388 76.2 90)
 			(hide yes)
@@
 			)
 		)
-		(property "Value" "6,8n"
+		(property "Value" "6.8n"
 			(at 83.82 160.782 0)
 			(show_name no)
@@
 			)
 		)
-		(property "Footprint" "Capacitor_SMD:C_0603_1608Metric_Pad1.08x0.95mm_HandSolder"
+		(property "Footprint" "Capacitor_SMD:C_0603_1608Metric"
 			(at 78.74 158.4452 0)
 			(hide yes)
@@
 			)
 		)
-		(property "Footprint" "Capacitor_SMD:C_1206_3216Metric_Pad1.33x1.80mm_HandSolder"
+		(property "Footprint" "Capacitor_SMD:C_1206_3216Metric"
 			(at 237.49 140.0048 0)
 			(hide yes)
